Commit message: pi tweaks

File: xavbot_description/urdf/xavbot.platform.ros2_control.xacro (robot description, xacro)
@@ -10,10 +10,10 @@
         <param name="rr_name">rear_right_wheel_joint</param>
         <param name="fl_port">1</param>
-        <param name="fr_port">0</param>
-        <param name="rl_port">2</param>
+        <param name="fr_port">2</param>
+        <param name="rl_port">0</param>
         <param name="rr_port">3</param>
         <param name="fl_direction">-1</param>
-        <param name="fr_direction">-1</param>
-        <param name="rl_direction">1</param>
+        <param name="fr_direction">1</param>
+        <param name="rl_direction">-1</param>
         <param name="rr_direction">1</param>
         <param name="device">/dev/ttyACM0</param>

File: xavbot_description/urdf/xavbot.urdf.xacro (robot description, xacro)
@@ -11,5 +11,5 @@
   </xacro:sensor_d435i>
   <xacro:sensor_d435i parent="base_link" name="arm_camera" use_nominal_extrinsics="false">
-    <origin xyz="0.173 0.13 0.163" rpy="0 0.7854 0"/>
+    <origin xyz="0.173 0.13 0.163" rpy="0 0.6981 0"/>
   </xacro:sensor_d435i>
   <!-- Import xavbot ros2_control description -->

Commit message: Swap to official mecanum controller

File: xavbot_description/urdf/xavbot.platform.ros2_control.xacro (robot description, xacro)
@@ -9,10 +9,10 @@
         <param name="rl_name">rear_left_wheel_joint</param>
         <param name="rr_name">rear_right_wheel_joint</param>
-        <param name="fl_port">1</param>
+        <param name="fl_port">0</param>
         <param name="fr_port">2</param>
-        <param name="rl_port">0</param>
+        <param name="rl_port">1</param>
         <param name="rr_port">3</param>
-        <param name="fl_direction">1</param>
-        <param name="fr_direction">-1</param>
+        <param name="fl_direction">-1</param>
+        <param name="fr_direction">1</param>
         <param name="rl_direction">-1</param>
         <param name="rr_direction">1</param>

File: xavbot_description/urdf/xavbot.platform.xacro (robot description, xacro)
@@ -11,5 +11,4 @@
     <xacro:property name="wheel_length" value="0.024" />
     <xacro:property name="wheel_radius" value="0.0185" />
-    <xacro:property name="profile_size" value="0.02" />
     <!-- Base Link -->
     <link name="${prefix}base_link">
