Commit message: Update arm urdf

File: xavbot_description/urdf/xavbot.arm.urdf.xacro (robot description, xacro)
@@ -1,15 +1,10 @@
 <?xml version="1.0"?>
-<robot xmlns:xacro="http://www.ros.org/wiki/xacro" name="xavbot">
+<robot xmlns:xacro="http://www.ros.org/wiki/xacro" name="xavbot_arm">
   <xacro:arg name="prefix" default="" />
-  <xacro:arg name="standalone" default="true" />
   <!-- Import Geometry -->
   <xacro:include filename="$(find xavbot_description)/urdf/xavbot.arm.xacro" />
-  <xacro:xavbot_arm prefix="$(arg prefix)" mesh_dir="package://xavbot_description/meshes" standalone="$(arg standalone)" />
+  <xacro:xavbot_arm prefix="$(arg prefix)" mesh_dir="package://xavbot_description/meshes" standalone="true" />
   <!-- Import xavbot ros2_control description -->
   <xacro:include filename="$(find xavbot_description)/urdf/xavbot.arm.ros2_control.xacro" />
-  <xacro:xavbot_arm_control name="xavbot" prefix="$(arg prefix)" />
-  <!-- Import Rviz colors -->
-  <xacro:if value="$(arg standalone)">
-    <xacro:include filename="$(find xavbot_description)/urdf/xavbot.materials.xacro" />
-  </xacro:if>
+  <xacro:xavbot_arm_control name="xavbot_arm" prefix="$(arg prefix)" />
 </robot>

File: xavbot_description/urdf/xavbot.arm.xacro (robot description, xacro)
@@ -10,5 +10,5 @@
           <parent link="${prefix}base_link"/>
           <child link="${prefix}link0"/>
-          <origin xyz="0 0 0" rpy="${PI/2} 0 ${PI}"/>
+          <origin xyz="0 0 0" rpy="0 0 0"/>
         </joint>
       </xacro:if>
@@ -17,12 +17,12 @@
           <parent link="${prefix}base_link"/>
           <child link="${prefix}link0"/>
-          <origin xyz="0.18 0.180 0.073" rpy="${PI/2} 0 ${PI}"/>
+          <origin xyz="0.18 0.180 0.073" rpy="0 0 0"/>
         </joint>
       </xacro:unless>
       <link name="${prefix}link0">
         <collision>
-          <origin xyz="0 0 0" rpy="0 0 0"/>
+          <origin xyz="0 0 0.02325" rpy="0 0 0"/>
           <geometry>
-            <mesh filename="${mesh_dir}/collision/link0.stl" scale="0.001 0.001 0.001"/>
+            <box size="0.0285 0.04 0.0465"/>
           </geometry>
         </collision>
@@ -30,16 +30,7 @@
           <origin xyz="0 0 0" rpy="0 0 0"/>
           <geometry>
-            <mesh filename="${mesh_dir}/visual/link0.stl" scale="0.001 0.001 0.001"/>
+            <mesh filename="${mesh_dir}/link0.dae" scale="1 1 1"/>
           </geometry>
-          <material name="grey"/>
         </visual>
-        <inertial>
-          <origin xyz="0 -0.013 0" rpy="0 0 0"/>
-          <mass value="0.0572"/>
-          <inertia
-            ixx="${0.0572 / 12.0 * (0.0465*0.0465 + 0.034*0.034)}" ixy="0.0" ixz="0.0"
-            iyy="${0.0572 / 12.0 * (0.034*0.034 + 0.0285*0.0285)}" iyz="0.0"
-            izz="${0.0572 / 12.0 * (0.0285*0.0285 + 0.0465*0.0465)}"/>
-        </inertial>
       </link>
       <!-- link1 -->
@@ -47,5 +38,5 @@
         <parent link="${prefix}link0"/>
         <child link="${prefix}link1"/>
-        <origin xyz="0 0 0" rpy="0 0 0"/>
+        <origin xyz="0 0 0.03525" rpy="${PI / 2} 0 0"/>
         <axis xyz="0 0 1"/>
         <dynamics damping="0.2"/>
@@ -59,24 +50,15 @@
       <link name="${prefix}link1">
         <collision>
-          <origin xyz="0 0 0" rpy="0 0 0"/>
+          <origin xyz="0 0.0585 0" rpy="0 0 0"/>
           <geometry>
-            <mesh filename="${mesh_dir}/collision/link1.stl" scale="0.001 0.001 0.001"/>
+            <box size="0.0285 0.1455 0.044"/>
           </geometry>
         </collision>
         <visual>
-          <origin xyz="0 0 0" rpy="0 0 0"/>
+          <origin xyz="0 0 0" rpy="0 ${PI} 0"/>
           <geometry>
-            <mesh filename="${mesh_dir}/visual/link1.stl" scale="0.001 0.001 0.001"/>
+            <mesh filename="${mesh_dir}/link1.dae" scale="1 1 1"/>
           </geometry>
-          <material name="grey"/>
         </visual>
-        <inertial>
-          <origin xyz="0 -0.013 0" rpy="0 0 0"/>
-          <mass value="0.0572"/>
-          <inertia
-            ixx="${0.0572 / 12.0 * (0.0465*0.0465 + 0.034*0.034)}" ixy="0.0" ixz="0.0"
-            iyy="${0.0572 / 12.0 * (0.034*0.034 + 0.0285*0.0285)}" iyz="0.0"
-            izz="${0.0572 / 12.0 * (0.0285*0.0285 + 0.0465*0.0465)}"/>
-        </inertial>
       </link>
       <!-- link2 -->
@@ -84,35 +66,6 @@
         <parent link="${prefix}link1"/>
         <child link="${prefix}link2"/>
-        <origin xyz="0 0.1 0" rpy="0 0 0"/>
+        <origin xyz="0 0.12 0" rpy="0 0 0"/>
         <axis xyz="0 0 1"/>
-        <dynamics damping="0.2"/>
-        <limit
-          lower="${-8 * PI/9}"
-          upper="${PI/2}"
-          effort="4.0"
-          velocity="5.5">
-        </limit>
-      </joint>
-      <link name="${prefix}link2">
-        <collision>
-          <origin xyz="0 0 0" rpy="0 0 0"/>
-          <geometry>
-            <mesh filename="${mesh_dir}/collision/link2.stl" scale="0.001 0.001 0.001"/>
-          </geometry>
-        </collision>
-        <visual>
-          <origin xyz="0 0 0" rpy="0 0 0"/>
-          <geometry>
-            <mesh filename="${mesh_dir}/visual/link2.stl" scale="0.001 0.001 0.001"/>
-          </geometry>
-          <material name="grey"/>
-        </visual>
-      </link>
-      <!-- link3 -->
-      <joint name="${prefix}link3_joint" type="revolute">
-        <parent link="${prefix}link2"/>
-        <child link="${prefix}link3"/>
-        <origin xyz="-0.1 0.04 0" rpy="0 0 0"/>
-        <axis xyz="0 0 1 "/>
         <dynamics damping="0.2"/>
         <limit
@@ -123,9 +76,49 @@
         </limit>
       </joint>
+      <link name="${prefix}link2">
+        <collision>
+          <origin xyz="0 0.015 0" rpy="0 0 0"/>
+          <geometry>
+            <box size="0.0285 0.0585 0.044"/>
+          </geometry>
+        </collision>
+          <collision>
+          <origin xyz="0.0535 0.03 0" rpy="0 0 0"/>
+          <geometry>
+            <box size="0.1355 0.0285 0.044"/>
+          </geometry>
+        </collision>
+        <visual>
+          <origin xyz="0 0 0" rpy="0 ${PI} 0"/>
+          <geometry>
+            <mesh filename="${mesh_dir}/link2.dae" scale="1 1 1"/>
+          </geometry>
+        </visual>
+      </link>
+      <!-- link3 -->
+      <joint name="${prefix}link3_joint" type="revolute">
+        <parent link="${prefix}link2"/>
+        <child link="${prefix}link3"/>
+        <origin xyz="0.11 0.03 0" rpy="0 0 ${-PI/2}"/>
+        <axis xyz="0 0 -1 "/>
+        <dynamics damping="0.2"/>
+        <limit
+          lower="-${PI/2}"
+          upper="${PI/2}"
+          effort="4.0"
+          velocity="5.5">
+        </limit>
+      </joint>
       <link name="${prefix}link3">
         <collision>
-          <origin xyz="0 0 0" rpy="0 0 0"/>
+          <origin xyz="0 0.016875 0" rpy="0 0 0"/>
           <geometry>
-            <mesh filename="${mesh_dir}/collision/link3.stl" scale="0.001 0.001 0.001"/>
+            <box size="0.0285 0.06225 0.044"/>
+          </geometry>
+        </collision>
+        <collision>
+          <origin xyz="0 0.0535 -0.0075" rpy="0 0 0"/>
+          <geometry>
+            <box size="0.01 0.011 0.1"/>
           </geometry>
         </collision>
@@ -133,115 +126,70 @@
           <origin xyz="0 0 0" rpy="0 0 0"/>
           <geometry>
-            <mesh filename="${mesh_dir}/visual/link3.stl" scale="0.001 0.001 0.001"/>
+            <mesh filename="${mesh_dir}/link3.dae" scale="1 1 1"/>
           </geometry>
-          <material name="grey"/>
         </visual>
       </link>
-      <!-- link4 -->
-      <joint name="${prefix}link4_joint" type="revolute">
+      <!-- gripper_virtual -->
+      <link name="${prefix}gripper_virtual"/>
+      <joint name="${prefix}gripper_virtual_joint" type="prismatic">
         <parent link="${prefix}link3"/>
-        <child link="${prefix}link4"/>
-        <origin xyz="-0.061 0 0" rpy="0 ${-PI/2} 0"/>
-        <axis xyz="0 0 1"/>
-        <dynamics damping="0.2"/>
+        <child link="${prefix}gripper_virtual"/>
+        <origin xyz="0 0 0" rpy="0 0 ${PI/2}"/>
+        <axis xyz="1 0 0"/>
         <limit
-          lower="-${PI}"
-          upper="${PI}"
+          lower="0.0"
+          upper="0.0536"
           effort="4.0"
-          velocity="5.5">
-        </limit>
+          velocity="0.1"/>
       </joint>
-      <link name="${prefix}link4">
+      <!-- gripper_tcp -->
+      <link name="${prefix}gripper_tcp"/>
+      <joint name="${prefix}gripper_tcp_joint" type="fixed">
+        <parent link="${prefix}link3"/>
+        <child link="${prefix}gripper_tcp"/>
+        <origin xyz="0 0.105 -0.0075" rpy="${-PI/2} 0 ${PI/2}"/>
+      </joint>
+      <!-- rightfinger -->
+      <joint name="${prefix}rightfinger_joint" type="prismatic">
+        <parent link="${prefix}link3"/>
+        <child link="${prefix}rightfinger"/>
+        <mimic joint="${prefix}gripper_virtual_joint" multiplier="0.5"/>
+        <origin xyz="0 0.059 0.00375" rpy="${-PI/2} ${-PI/2} 0"/>
+        <axis xyz="0 0 1 "/>
+      </joint>
+      <link name="${prefix}rightfinger">
         <collision>
-          <origin xyz="0 0 0" rpy="0 0 0"/>
+          <origin xyz="-0.00975 0 0.02657" rpy="0 0 0"/>
           <geometry>
-            <mesh filename="${mesh_dir}/collision/link4.stl" scale="0.001 0.001 0.001"/>
+            <box size="0.003 0.017 0.05314"/>
           </geometry>
         </collision>
         <visual>
-          <origin xyz="0 0 0" rpy="0 0 0"/>
+          <origin xyz="0 0 0" rpy="0 0 ${-PI/2}"/>
           <geometry>
-            <mesh filename="${mesh_dir}/visual/link4.stl" scale="0.001 0.001 0.001"/>
+            <mesh filename="${mesh_dir}/finger.dae" scale="1 1 1"/>
           </geometry>
-          <material name="grey"/>
-        </visual>
-      </link>
-      <!-- hand_tcp -->
-      <joint name="${prefix}tcp_joint" type="fixed">
-        <parent link="${prefix}link4"/>
-        <child link="${prefix}tcp"/>
-        <origin xyz="0 0 0.08" rpy="${PI/2} ${-PI/2} 0"/>
-      </joint>
-      <link name="${prefix}tcp"/>
-      <!-- gripper_crank -->
-      <joint name="${prefix}gripper_joint" type="revolute">
-        <parent link="${prefix}link4"/>
-        <child link="${prefix}gripper_crank"/>
-        <origin xyz="0 0 0.04" rpy="0 0 0"/>
-        <axis xyz="0 0 1"/>
-        <limit
-          lower="0"
-          upper="1.047"
-          effort="4.0"
-          velocity="5.5">
-        </limit>
-      </joint>
-      <link name="${prefix}gripper_crank"/>
-      <!-- rightfinger -->
-      <joint name="${prefix}rightfinger_joint" type="prismatic">
-        <parent link="${prefix}link4"/>
-        <child link="${prefix}rightfinger"/>
-        <origin xyz="0 0 0.045" rpy="0 0 0"/>
-        <axis xyz="-1 0 0"/>
-        <limit
-          lower="0"
-          upper="0.0265"
-          effort="9.9"
-          velocity="9.9">
-        </limit>
-        <mimic joint="${prefix}gripper_joint" multiplier="0.024446"/>
-      </joint>
-      <link name="${prefix}rightfinger">
-        <collision>
-          <origin xyz="0 0 0" rpy="0 0 0"/>
-          <geometry>
-            <mesh filename="${mesh_dir}/collision/finger.stl" scale="0.001 0.001 0.001"/>
-          </geometry>
-        </collision>
-        <visual>
-          <origin xyz="0 0 0" rpy="0 0 0"/>
-          <geometry>
-            <mesh filename="${mesh_dir}/visual/finger.stl" scale="0.001 0.001 0.001"/>
-          </geometry>
-          <material name="grey"/>
         </visual>
       </link>
       <!-- leftfinger -->
       <joint name="${prefix}leftfinger_joint" type="prismatic">
-        <parent link="${prefix}link4"/>
+        <parent link="${prefix}link3"/>
         <child link="${prefix}leftfinger"/>
-        <origin xyz="0 0 0.045" rpy="0 0 ${PI}"/>
-        <axis xyz="-1 0 0"/>
-        <limit
-          lower="0"
-          upper="0.0265"
-          effort="9.9"
-          velocity="9.9">
-        </limit>
-        <mimic joint="${prefix}gripper_joint" multiplier="0.024446"/>
+        <mimic joint="${prefix}gripper_virtual_joint" multiplier="0.5"/>
+        <origin xyz="0 0.059 -0.01875" rpy="${-PI/2} ${PI/2} 0"/>
+        <axis xyz="0 0 1 "/>
       </joint>
       <link name="${prefix}leftfinger">
         <collision>
-          <origin xyz="0 0 0" rpy="0 0 0"/>
+          <origin xyz="-0.00975 0 0.02657" rpy="0 0 0"/>
           <geometry>
-            <mesh filename="${mesh_dir}/collision/finger.stl" scale="0.001 0.001 0.001"/>
+            <box size="0.003 0.017 0.05314"/>
           </geometry>
         </collision>
         <visual>
-          <origin xyz="0 0 0" rpy="0 0 0"/>
+          <origin xyz="0 0 0" rpy="0 0 ${-PI/2}"/>
           <geometry>
-            <mesh filename="${mesh_dir}/visual/finger.stl" scale="0.001 0.001 0.001"/>
+            <mesh filename="${mesh_dir}/finger.dae" scale="1 1 1"/>
           </geometry>
-          <material name="grey"/>
         </visual>
       </link>

File: xavbot_description/urdf/xavbot.platform.xacro (robot description, xacro)
@@ -34,5 +34,5 @@
         <origin xyz="0 0 ${wheel_radius}" rpy="0 0 0"/>
         <geometry>
-          <mesh filename="${mesh_dir}/visual/xavbot_chassis_2.1.0.dae"/>
+          <mesh filename="${mesh_dir}/xavbot_chassis_2.1.0.dae"/>
         </geometry>
       </visual>
@@ -55,5 +55,5 @@
         <origin xyz="0 0 0" rpy="0 0 0"/>
         <geometry>
-          <mesh filename="${mesh_dir}/visual/mecanum_simple.dae"/>
+          <mesh filename="${mesh_dir}/mecanum_simple.dae"/>
         </geometry>
       </visual>
@@ -76,5 +76,5 @@
         <origin xyz="0 0 0" rpy="0 0 0"/>
         <geometry>
-          <mesh filename="${mesh_dir}/visual/mecanum_simple.dae"/>
+          <mesh filename="${mesh_dir}/mecanum_simple.dae"/>
         </geometry>
       </visual>
@@ -97,5 +97,5 @@
         <origin xyz="0 0 0" rpy="0 0 0"/>
         <geometry>
-          <mesh filename="${mesh_dir}/visual/mecanum_simple.dae"/>
+          <mesh filename="${mesh_dir}/mecanum_simple.dae"/>
         </geometry>
       </visual>
@@ -118,5 +118,5 @@
         <origin xyz="0 0 0" rpy="0 0 0"/>
         <geometry>
-          <mesh filename="${mesh_dir}/visual/mecanum_simple.dae"/>
+          <mesh filename="${mesh_dir}/mecanum_simple.dae"/>
         </geometry>
       </visual>

File: xavbot_description/urdf/xavbot.urdf.xacro (robot description, xacro)
@@ -2,5 +2,5 @@
 <robot xmlns:xacro="http://www.ros.org/wiki/xacro" name="xavbot">
   <xacro:arg name="prefix" default="" />
-  <xacro:arg name="arm" default="false" />
+  <xacro:arg name="arm" default="true" />
   <!-- Import Geometry -->
   <xacro:include filename="$(find xavbot_description)/urdf/xavbot.platform.xacro" />
