Commit message: Update URDF

File: xavbot_description/urdf/xavbot.arm.xacro (robot description, xacro)
@@ -17,5 +17,5 @@
           <parent link="${prefix}base_link"/>
           <child link="${prefix}link0"/>
-          <origin xyz="0.210 0.200 0.073" rpy="${PI/2} 0 ${PI}"/>
+          <origin xyz="0.18 0.180 0.073" rpy="${PI/2} 0 ${PI}"/>
         </joint>
       </xacro:unless>

File: xavbot_description/urdf/xavbot.platform.xacro (robot description, xacro)
@@ -5,7 +5,7 @@
     <xacro:property name="PI" value="3.1415926535897931"/>
     <xacro:property name="base_mass" value="1.0" /> <!-- arbitrary value for base mass -->
-    <xacro:property name="base_width" value="0.21" />
-    <xacro:property name="base_length" value="0.22" />
-    <xacro:property name="base_height" value="0.07" />
+    <xacro:property name="base_width" value="0.22" />
+    <xacro:property name="base_length" value="0.21" />
+    <xacro:property name="base_height" value="0.05" />
     <xacro:property name="wheel_mass" value="0.02" /> <!-- arbitrary value for wheel mass -->
     <xacro:property name="wheel_length" value="0.024" />
@@ -15,8 +15,20 @@
     <link name="${prefix}base_link">
       <collision>
-        <origin xyz="${base_length / 2} ${base_width / 2} ${wheel_radius + 0.009}" rpy="0 0 0"/>
+        <origin xyz="${base_length / 2} ${base_width / 2} ${wheel_radius + 0.005}" rpy="0 0 0"/>
         <geometry>
-          <box size="${base_length} ${base_width} ${base_height}"/>
+          <box size="${base_length} ${base_width} ${2 * wheel_radius + 0.01}"/>
         </geometry>
+      </collision>
+      <collision>
+        <origin xyz="0.095 0.08 0.06" rpy="0 0 0"/>
+          <geometry>
+            <box size="0.16 0.16 0.025"/>
+          </geometry>
+      </collision>
+      <collision>
+        <origin xyz="0.075 0.08 0.1125" rpy="0 0 0"/>
+          <geometry>
+            <box size="0.12 0.16 0.08"/>
+          </geometry>
       </collision>
       <visual>
@@ -36,5 +48,5 @@
     <link name="${prefix}front_left_wheel">
       <collision>
-        <origin xyz="0 0 0" rpy="0 0 0"/>
+        <origin xyz="0 0 ${wheel_length / 2}" rpy="0 0 0"/>
         <geometry>
           <cylinder radius="${wheel_radius}" length="${wheel_length}"/>
@@ -57,5 +69,5 @@
     <link name="${prefix}front_right_wheel">
       <collision>
-        <origin xyz="0 0 0" rpy="0 0 0"/>
+        <origin xyz="0 0 ${wheel_length / 2}" rpy="0 0 0"/>
         <geometry>
           <cylinder radius="${wheel_radius}" length="${wheel_length}"/>
@@ -78,5 +90,5 @@
     <link name="${prefix}rear_left_wheel">
       <collision>
-        <origin xyz="0 0 0" rpy="0 0 0"/>
+        <origin xyz="0 0 ${wheel_length / 2}" rpy="0 0 0"/>
         <geometry>
           <cylinder radius="${wheel_radius}" length="${wheel_length}"/>
@@ -99,5 +111,5 @@
     <link name="${prefix}rear_right_wheel">
       <collision>
-        <origin xyz="0 0 0" rpy="0 0 0"/>
+        <origin xyz="0 0 ${wheel_length / 2}" rpy="0 0 0"/>
         <geometry>
           <cylinder radius="${wheel_radius}" length="${wheel_length}"/>

File: xavbot_description/urdf/xavbot.urdf.xacro (robot description, xacro)
@@ -2,5 +2,5 @@
 <robot xmlns:xacro="http://www.ros.org/wiki/xacro" name="xavbot">
   <xacro:arg name="prefix" default="" />
-  <xacro:arg name="arm" default="true" />
+  <xacro:arg name="arm" default="false" />
   <!-- Import Geometry -->
   <xacro:include filename="$(find xavbot_description)/urdf/xavbot.platform.xacro" />
@@ -8,5 +8,5 @@
   <xacro:include filename="$(find realsense2_description)/urdf/_d435i.urdf.xacro"/>
   <xacro:sensor_d435i parent="base_link" name="VIO_camera" use_nominal_extrinsics="false">
-    <origin xyz="0.22425 0.14 0.09" rpy="0 0 0"/>
+    <origin xyz="0.129 0.08 0.0985" rpy="0 0 0"/>
   </xacro:sensor_d435i>
   <!-- Import xavbot ros2_control description -->
@@ -18,7 +18,4 @@
     <xacro:include filename="$(find xavbot_description)/urdf/xavbot.arm.xacro" />
     <xacro:xavbot_arm prefix="$(arg prefix)" mesh_dir="package://xavbot_description/meshes" standalone="false" />
-    <xacro:sensor_d435i parent="base_link" name="arm_camera" use_nominal_extrinsics="false">
-      <origin xyz="0.173 0.13 0.163" rpy="0 0.6981 0"/>
-    </xacro:sensor_d435i>
     <!-- Import xavbot ros2_control description -->
     <xacro:include filename="$(find xavbot_description)/urdf/xavbot.arm.ros2_control.xacro" />

Commit message: Update moveit config

File: xavbot_description/urdf/xavbot.arm.xacro (robot description, xacro)
@@ -17,5 +17,5 @@
           <parent link="${prefix}base_link"/>
           <child link="${prefix}link0"/>
-          <origin xyz="0.18 0.180 0.073" rpy="0 0 0"/>
+          <origin xyz="0.17925 0.186 0.05195" rpy="0 0 0"/>
         </joint>
       </xacro:unless>
@@ -139,5 +139,5 @@
         <limit
           lower="0.0"
-          upper="0.0536"
+          upper="0.055"
           effort="4.0"
           velocity="0.1"/>
@@ -156,5 +156,10 @@
         <mimic joint="${prefix}gripper_virtual_joint" multiplier="0.5"/>
         <origin xyz="0 0.059 0.00375" rpy="${-PI/2} ${-PI/2} 0"/>
-        <axis xyz="0 0 1 "/>
+        <axis xyz="1 0 0 "/>
+        <limit
+          lower="0.0"
+          upper="0.0275"
+          velocity="0.05"
+          effort="2.0"/>
       </joint>
       <link name="${prefix}rightfinger">
@@ -178,5 +183,10 @@
         <mimic joint="${prefix}gripper_virtual_joint" multiplier="0.5"/>
         <origin xyz="0 0.059 -0.01875" rpy="${-PI/2} ${PI/2} 0"/>
-        <axis xyz="0 0 1 "/>
+        <axis xyz="1 0 0 "/>
+        <limit
+          lower="0.0"
+          upper="0.0275"
+          velocity="0.05"
+          effort="2.0"/>
       </joint>
       <link name="${prefix}leftfinger">

File: xavbot_description/urdf/xavbot.platform.xacro (robot description, xacro)
@@ -32,7 +32,7 @@
       </collision>
       <visual>
-        <origin xyz="0 0 ${wheel_radius}" rpy="0 0 0"/>
+        <origin xyz="0 0 ${wheel_radius + 0.00495} " rpy="0 0 0"/>
         <geometry>
-          <mesh filename="${mesh_dir}/xavbot_chassis_2.1.0.dae"/>
+          <mesh filename="${mesh_dir}/base.dae"/>
         </geometry>
       </visual>

File: xavbot_moveit_config/config/xavbot.ros2_control.xacro (robot description, xacro)
@@ -10,4 +10,5 @@
             <joint name="link1_joint">
                 <command_interface name="position"/>
+                <command_interface name="velocity"/>
                 <state_interface name="position">
                   <param name="initial_value">${initial_positions['link1_joint']}</param>
@@ -17,4 +18,5 @@
             <joint name="link2_joint">
                 <command_interface name="position"/>
+                <command_interface name="velocity"/>
                 <state_interface name="position">
                   <param name="initial_value">${initial_positions['link2_joint']}</param>
@@ -24,4 +26,5 @@
             <joint name="link3_joint">
                 <command_interface name="position"/>
+                <command_interface name="velocity"/>
                 <state_interface name="position">
                   <param name="initial_value">${initial_positions['link3_joint']}</param>
@@ -29,15 +32,17 @@
                 <state_interface name="velocity"/>
             </joint>
-            <joint name="link4_joint">
+            <joint name="gripper_virtual_joint">
                 <command_interface name="position"/>
+                <command_interface name="velocity"/>
                 <state_interface name="position">
-                  <param name="initial_value">${initial_positions['link4_joint']}</param>
+                  <param name="initial_value">${initial_positions['gripper_virtual_joint']}</param>
                 </state_interface>
                 <state_interface name="velocity"/>
             </joint>
-            <joint name="gripper_joint">
+            <joint name="virtual_joint">
                 <command_interface name="position"/>
+                <command_interface name="velocity"/>
                 <state_interface name="position">
-                  <param name="initial_value">${initial_positions['gripper_joint']}</param>
+                  <param name="initial_value">${initial_positions['virtual_joint']}</param>
                 </state_interface>
                 <state_interface name="velocity"/>

File: xavbot_moveit_config/config/xavbot.urdf.xacro (robot description, xacro)
@@ -6,4 +6,4 @@
     <!-- Import control_xacro -->
     <xacro:include filename="xavbot.ros2_control.xacro" />
-    <!-- <xacro:xavbot_ros2_control name="FakeSystem" initial_positions_file="$(arg initial_positions_file)"/> -->
+    <xacro:xavbot_ros2_control name="FakeSystem" initial_positions_file="$(arg initial_positions_file)"/>
 </robot>

Commit message: Move base_link to centre

File: xavbot_description/urdf/xavbot.arm.xacro (robot description, xacro)
@@ -17,5 +17,5 @@
           <parent link="${prefix}base_link"/>
           <child link="${prefix}link0"/>
-          <origin xyz="0.17925 0.186 0.05195" rpy="0 0 0"/>
+          <origin xyz="0.07425 0.076 0.05195" rpy="0 0 0"/>
         </joint>
       </xacro:unless>

File: xavbot_description/urdf/xavbot.platform.xacro (robot description, xacro)
@@ -11,8 +11,10 @@
     <xacro:property name="wheel_length" value="0.024" />
     <xacro:property name="wheel_radius" value="0.0185" />
+    <xacro:property name="half_width" value="${base_width / 2}" />
+    <xacro:property name="half_length" value="${base_length / 2}" />
     <!-- Base Link -->
     <link name="${prefix}base_link">
       <collision>
-        <origin xyz="${base_length / 2} ${base_width / 2} ${wheel_radius + 0.005}" rpy="0 0 0"/>
+        <origin xyz="0 0 ${wheel_radius + 0.00495}" rpy="0 0 0"/>
         <geometry>
           <box size="${base_length} ${base_width} ${2 * wheel_radius + 0.01}"/>
@@ -32,5 +34,5 @@
       </collision>
       <visual>
-        <origin xyz="0 0 ${wheel_radius + 0.00495} " rpy="0 0 0"/>
+        <origin xyz="${-half_length} ${-half_width} ${wheel_radius + 0.00495} " rpy="0 0 0"/>
         <geometry>
           <mesh filename="${mesh_dir}/base.dae"/>
@@ -42,5 +44,5 @@
       <parent link="${prefix}base_link"/>
       <child link="${prefix}front_left_wheel"/>
-      <origin xyz="${base_length - 0.03} ${base_width} ${wheel_radius}" rpy="-${PI/2} ${PI} 0"/>
+      <origin xyz="${half_length - 0.03} ${half_width} ${wheel_radius}" rpy="-${PI/2} ${PI} 0"/>
       <axis xyz="0 0 1"/>
     </joint>
@@ -63,5 +65,5 @@
       <parent link="${prefix}base_link"/>
       <child link="${prefix}front_right_wheel"/>
-      <origin xyz="${base_length - 0.03} 0 ${wheel_radius}" rpy="${PI/2} 0 0"/>
+      <origin xyz="${half_length - 0.03} ${-half_width} ${wheel_radius}" rpy="${PI/2} 0 0"/>
       <axis xyz="0 0 -1"/>
     </joint>
@@ -84,5 +86,5 @@
       <parent link="${prefix}base_link"/>
       <child link="${prefix}rear_left_wheel"/>
-      <origin xyz="0.03 ${base_width} ${wheel_radius}" rpy="-${PI/2} ${PI} 0"/>
+      <origin xyz="${-half_length + 0.03} ${half_width} ${wheel_radius}" rpy="-${PI/2} ${PI} 0"/>
       <axis xyz="0 0 1"/>
     </joint>
@@ -105,5 +107,5 @@
       <parent link="${prefix}base_link"/>
       <child link="${prefix}rear_right_wheel"/>
-      <origin xyz="0.03 0 ${wheel_radius}" rpy="${PI/2} 0 0"/>
+      <origin xyz="${-half_length + 0.03} ${-half_width} ${wheel_radius}" rpy="${PI/2} 0 0"/>
       <axis xyz="0 0 -1"/>
     </joint>

File: xavbot_description/urdf/xavbot.urdf.xacro (robot description, xacro)
@@ -8,5 +8,5 @@
   <xacro:include filename="$(find realsense2_description)/urdf/_d435i.urdf.xacro"/>
   <xacro:sensor_d435i parent="base_link" name="VIO_camera" use_nominal_extrinsics="false">
-    <origin xyz="0.129 0.08 0.0985" rpy="0 0 0"/>
+    <origin xyz="0.024 -0.03 0.0985" rpy="0 0 0"/>
   </xacro:sensor_d435i>
   <!-- Import xavbot ros2_control description -->
