Commit message: Real moveit working

File: xavbot_description/urdf/xavbot.arm.ros2_control.xacro (robot description, xacro)
@@ -2,50 +2,105 @@
 <robot xmlns:xacro="http://www.ros.org/wiki/xacro">
   <xacro:macro name="xavbot_arm_control" params="name prefix">
+    <xacro:property name="PI" value="3.1415926535897931"/>
     <ros2_control name="${name}" type="system">
       <hardware>
-        <plugin>dynamixel_hardware/DynamixelHardware</plugin>
-        <param name="usb_port">/dev/ttyUSB0</param>
+        <plugin>dynamixel_hardware_interface/DynamixelHardware</plugin>
+        <param name="port_name">/dev/ttyUSB0</param>
         <param name="baud_rate">57600</param>
+        <param name="error_timeout_ms">10000</param>
+        <param name="dynamixel_model_folder">/param/dxl_model</param>
+        <param name="number_of_joints">4</param>
+        <param name="number_of_transmissions">4</param>
+        <param name="disable_torque_at_init">false</param>
+        <param name="transmission_to_joint_matrix">
+          1, 0, 0, 0,
+          0, 1, 0, 0,
+          0, 0, 1, 0,
+          0, 0, 0, 1
+        </param>
+        <param name="joint_to_transmission_matrix">
+          1, 0, 0, 0,
+          0, 1, 0, 0,
+          0, 0, 1, 0,
+          0, 0, 0, 1
+        </param>
+        <param name="use_revolute_to_prismatic_gripper">1</param>
+        <param name="revolute_to_prismatic_dxl">dxl4</param>
+        <param name="revolute_max">${PI / 3}</param>
+        <param name="revolute_min">0.0</param>
+        <param name="revolute_to_prismatic_joint">${prefix}gripper_virtual_joint</param>
+        <param name="prismatic_max">0.0275</param>
+        <param name="prismatic_min">0.0</param>
       </hardware>
       <joint name="${prefix}link1_joint">
-        <param name="id">10</param>
         <command_interface name="position"/>
         <command_interface name="velocity"/>
         <state_interface name="position"/>
         <state_interface name="velocity"/>
-        <state_interface name="effort"/>
       </joint>
       <joint name="${prefix}link2_joint">
-        <param name="id">11</param>
         <command_interface name="position"/>
         <command_interface name="velocity"/>
         <state_interface name="position"/>
         <state_interface name="velocity"/>
-        <state_interface name="effort"/>
       </joint>
       <joint name="${prefix}link3_joint">
-        <param name="id">12</param>
         <command_interface name="position"/>
         <command_interface name="velocity"/>
         <state_interface name="position"/>
         <state_interface name="velocity"/>
-        <state_interface name="effort"/>
       </joint>
-      <joint name="${prefix}link4_joint">
-        <param name="id">13</param>
+      <joint name="${prefix}gripper_virtual_joint">
         <command_interface name="position"/>
         <command_interface name="velocity"/>
+        <command_interface name="effort"/>
         <state_interface name="position"/>
         <state_interface name="velocity"/>
         <state_interface name="effort"/>
       </joint>
-      <joint name="${prefix}gripper_joint">
-        <param name="id">14</param>
-        <command_interface name="position"/>
-        <command_interface name="velocity"/>
-        <state_interface name="position"/>
-        <state_interface name="velocity"/>
-        <state_interface name="effort"/>
-      </joint>
+      <gpio name="dxl1">
+        <param name="type">dxl</param>
+        <param name="ID">10</param>
+        <command_interface name="Goal Position"/>
+        <command_interface name="Goal Velocity"/>
+        <state_interface name="Present Position"/>
+        <state_interface name="Present Velocity"/>
+        <param name="Drive Mode">1</param>
+        <param name="Homing Offset">0</param>
+        <param name="Return Delay Time">50</param>
+      </gpio>
+      <gpio name="dxl2">
+        <param name="type">dxl</param>
+        <param name="ID">11</param>
+        <command_interface name="Goal Position"/>
+        <command_interface name="Goal Velocity"/>
+        <state_interface name="Present Position"/>
+        <state_interface name="Present Velocity"/>
+        <param name="Drive Mode">1</param>
+        <param name="Homing Offset">0</param>
+        <param name="Return Delay Time">50</param>
+      </gpio>
+      <gpio name="dxl3">
+        <param name="type">dxl</param>
+        <param name="ID">12</param>
+        <command_interface name="Goal Position"/>
+        <command_interface name="Goal Velocity"/>
+        <state_interface name="Present Position"/>
+        <state_interface name="Present Velocity"/>
+        <param name="Drive Mode">0</param>
+        <param name="Homing Offset">0</param>
+        <param name="Return Delay Time">50</param>
+      </gpio>
+      <gpio name="dxl4">
+        <param name="type">dxl</param>
+        <param name="ID">13</param>
+        <command_interface name="Goal Position"/>
+        <command_interface name="Goal Current"/>
+        <state_interface name="Present Position"/>
+        <state_interface name="Present Current"/>
+        <param name="Drive Mode">0</param>
+        <param name="Homing Offset">0</param>
+        <param name="Return Delay Time">50</param>
+      </gpio>
     </ros2_control>
   </xacro:macro>

File: xavbot_description/urdf/xavbot.platform.xacro (robot description, xacro)
@@ -22,5 +22,5 @@
       </collision>
       <collision>
-        <origin xyz="0.095 0.08 0.06" rpy="0 0 0"/>
+        <origin xyz="0 -0.03 0.06" rpy="0 0 0"/>
           <geometry>
             <box size="0.16 0.16 0.025"/>
@@ -28,5 +28,5 @@
       </collision>
       <collision>
-        <origin xyz="0.075 0.08 0.1125" rpy="0 0 0"/>
+        <origin xyz="0 -0.03 0.1125" rpy="0 0 0"/>
           <geometry>
             <box size="0.12 0.16 0.08"/>
